File: Schematic/HostInterface.kicad_sch (KiCad schematic)
At the start: 8 parts, among them U201 GAL22V10, U202 74LVC245, U203 74LVC245, U204 74LCV245

Commit message: change host bus signal names to match logic
This was a bit of a tedious change, but I think it's
worthwhile to make it more obvious how the logic
and schematic relate to each other.
Connections:
- net HostA0 renamed HostBusAddr0
- net HostA1 renamed HostBusAddr1
- net HostA10 renamed HostBusAddr10
- net HostA2 renamed HostBusAddr2
- net HostA3 renamed HostBusAddr3
- net HostA4 renamed HostBusAddr4
- net HostA5 renamed HostBusAddr5
- net HostA6 renamed HostBusAddr6
- net HostA7 renamed HostBusAddr7
- net HostA8 renamed HostBusAddr8
- net HostA9 renamed HostBusAddr9
- net HostD0 renamed HostBusData0
- net HostD1 renamed HostBusData1
- net HostD2 renamed HostBusData2
- net HostD3 renamed HostBusData3
- net HostD4 renamed HostBusData4
- net HostD5 renamed HostBusData5
- net HostD6 renamed HostBusData6
- net HostD7 renamed HostBusData7
