File: Schematic/HostInterface.kicad_sch (KiCad schematic)
At the start: 3 parts, among them U1 SN74LVC245APW, U2 SN74LVC245APW, U3 SN74LVC245APW

Commit message: done with host interface?
Parts:
- added C201, C202, C203: C, symbol Device:C
- renumbered U1 to U201, U2 to U202, U3 to U203
Connections:
- net GND: now also C201.2, C202.2, C203.2; no longer U203.9 (A8)
- net VCC: now also U202.1 (DIR), U203.1 (DIR), C201.1, C202.1, C203.1
- net ~{RST}: now reaches U203.11 (B8)
- new net Raw~{RST}: U203.9 (A8)
Other:
- note added: "Decoupling for U201-U203"
- moved on the sheet: U201, U202, U203
