File: Schematic/FPGA_VGA.kicad_sch (KiCad schematic)
At the start: 3 parts, among them U101 Upduino_3.0, Y101 25.175 MHz 7050 3.3V

Commit message: working on host interface / level translation
Other:
- added sheet HostInterface (HostInterface.kicad_sch)

Commit message: done with host interface?
Parts:
- added J1: Conn_01x08, symbol Connector_Generic:Conn_01x08
- added J2: Conn_01x13, symbol Connector_Generic:Conn_01x13
- added J3: Conn_01x03, symbol Connector_Generic:Conn_01x03
Connections:
- net HostInterface/RawHostA0: now also J2.1 (Pin_1)
- net HostInterface/RawHostA1: now also J2.2 (Pin_2)
- net HostInterface/RawHostA10: now also J2.11 (Pin_11)
- net HostInterface/RawHostA11: now also J2.12 (Pin_12)
- net HostInterface/RawHostA12: now also J2.13 (Pin_13)
- net HostInterface/RawHostA2: now also J2.3 (Pin_3)
- net HostInterface/RawHostA3: now also J2.4 (Pin_4)
- net HostInterface/RawHostA4: now also J2.5 (Pin_5)
- net HostInterface/RawHostA5: now also J2.6 (Pin_6)
- net HostInterface/RawHostA6: now also J2.7 (Pin_7)
- net HostInterface/RawHostA7: now also J2.8 (Pin_8)
- net HostInterface/RawHostA8: now also J2.9 (Pin_9)
- net HostInterface/RawHostA9: now also J2.10 (Pin_10)
- net HostInterface/RawHostD0: now also J1.1 (Pin_1)
- net HostInterface/RawHostD1: now also J1.2 (Pin_2)
- net HostInterface/RawHostD2: now also J1.3 (Pin_3)
- net HostInterface/RawHostD3: now also J1.4 (Pin_4)
- net HostInterface/RawHostD4: now also J1.5 (Pin_5)
- net HostInterface/RawHostD5: now also J1.6 (Pin_6)
- net HostInterface/RawHostD6: now also J1.7 (Pin_7)
- net HostInterface/RawHostD7: now also J1.8 (Pin_8)
- net HostInterface/Raw~{R}: now also J3.1 (Pin_1)
- net HostInterface/Raw~{W}: now also J3.2 (Pin_2)
- net -RST renamed ~{RST}
- new net HostInterface/Raw~{RST}: J3.3 (Pin_3)
Other:
- sheet HostInterface ports: added HostA0, HostA1, HostA10, HostA11, HostA12, HostA2, HostA3, HostA4, HostA5, HostA6, HostA7, HostA8, HostA9, HostD0, HostD1, HostD2, HostD3, HostD4, HostD5, HostD6, HostD7, Raw~{RST}, ~{RST}, ~{R}, ~{W}; removed none
- note added: "Signals from host system"
- moved on the sheet: U101, Y101
